Commit message: Fix IK elbow-up fallback and hand grasp-point geometry
- solve_ik: when the seed-continuity path (used during descent waypoints
  to avoid visible turning) lands on an unsafe elbow-down config with no
  other candidate, retry with the full seed list instead of accepting the
  unsafe pose. Confirmed live: the forearm was settling at -1.4cm (through
  the floor) on the final descent waypoint even though a safe elbow-up
  solution existed; continuity just never found it with only one seed to
  try.

- GRASP_POINT_IN_HAND_M: recomputed via FK sweep of the actual close-motion
  trajectory (real per-joint limits, not raw radians). The old point's Z
  was 7cm short of where any finger or thumb ever reaches while closing --
  confirmed live, only the pinky ever touched and the apple never left the
  table. New point is verified (offline FK) to put all four fingertips and
  the thumb within the apple's radius partway through their real close
  sweep.

- finger_alignment_node.py: lift() now IK-solves a real 15cm vertical wrist
  translation instead of a single shoulder_lift nudge (previously ~3cm).
  Added a ground-truth (ign topic, not vision) lift-hold check: pass only
  if the apple stays within 2cm horizontally and rises with the hand for
  3s. Fixed fingers-touched counting to count distinct fingers instead of
  per-joint hits (a single finger's 3 joints were being miscounted as "3
  fingers"), raised the lift-gate to >=2 distinct fingers + thumb, and
  added contact-link and fingertip-z-vs-apple-centroid logging.

- expanded_robot.urdf: regenerated from the current source xacros (mobile
  base self-collision removed, hand effort state interfaces) -- confirmed
  inert for the base_link-rooted IK chain this project actually uses.

File: vlm_scripts/expanded_robot.urdf (robot description, URDF)
Before this commit: robot mobile_ur, 41 links, 40 joints
Links:
- link mobile_base_link: geometry visual box size=0.36 0.36 0.25
Joints:
- joint caster_back_joint: origin xyz=-0.3 0 0.06 rpy=0 0 0 -> xyz=-0.16 0 0.06 rpy=0 0 0
- joint caster_front_joint: origin xyz=0.3 0 0.06 rpy=0 0 0 -> xyz=0.16 0 0.06 rpy=0 0 0
- joint left_wheel_joint: origin xyz=0 0.33 0.12 rpy=0 0 0 -> xyz=0 0.20 0.12 rpy=0 0 0
- joint right_wheel_joint: origin xyz=0 -0.33 0.12 rpy=0 0 0 -> xyz=0 -0.20 0.12 rpy=0 0 0
